File: pcb/RPi-Display_v10.brd (EAGLE design)
At the start: 85 x 56 mm, 42 parts, among them IC1 ADS7846, Q1 N-CHN, SW1 SW4S, U1 TS5204, X1 PASSER, X2 PASSER, X3 PASSER, X4 PASSER

Commit message: updated schematic and layout files
Parts:
- U1: value TS5204 -> TS5204-3V3
Routing:
- net N$7: track 0.00 -> 1.27 mm
Changed lines of the file:
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@@
 <?xml version="1.0" encoding="utf-8"?>
 <!DOCTYPE eagle SYSTEM "eagle.dtd">
-<eagle version="6.5.0">
+<eagle version="6.6.0">
 <drawing>
 <settings>
@@
 <attribute name="VALUE" x="54.9275" y="15.08125" size="0.8128" layer="28" font="vector" rot="MR90"/>
 </element>
-<element name="U1" library="Voltage-Reg" package="SOT23" value="TS5204" x="57.785" y="13.335" smashed="yes" rot="MR180">
+<element name="U1" library="Voltage-Reg" package="SOT23" value="TS5204-3V3" x="57.785" y="13.335" smashed="yes" rot="MR180">
 <attribute name="NAME" x="56.99125" y="11.27125" size="0.8128" layer="26" font="vector" ratio="10" rot="MR180"/>
 <attribute name="VALUE" x="57.4675" y="15.39875" size="0.8128" layer="28" font="vector" rot="MR90"/>
@@
 </signal>
 <signal name="N$3">
-<wire x1="52.07" y1="42.2275" x2="53.0225" y2="42.2275" width="0.254" layer="16"/>
+<wire x1="53.6575" y1="42.2275" x2="54.61" y2="42.2275" width="0.254" layer="16"/>
 </signal>
 <signal name="N$4">
-<wire x1="53.6575" y1="38.4175" x2="54.61" y2="38.4175" width="0.254" layer="16"/>
+<wire x1="52.07" y1="38.4175" x2="53.0225" y2="38.4175" width="0.254" layer="16"/>
 </signal>
 <signal name="IO22">
@@
 <wire x1="48.5775" y1="46.99" x2="48.5775" y2="47.9425" width="0.254" layer="16"/>
 </signal>
+<signal name="N$7">
+<wire x1="53.975" y1="32.385" x2="55.245" y2="32.385" width="0.254" layer="16"/>
+</signal>
 </signals>
