File: pcb/RPi-Display_Bplus_v10.brd (EAGLE design)
At the start: 69.5 x 56 mm, 56 parts, among them IC1 ADS7846, IC2 24LC-I/OT, Q1 N-CHN, SW1 SWITCH-PTS840P, SW2 SWITCH-PTS840P, SW3 SWITCH-PTS840P, U1 TS5204-3V3, X1 PASSER, X2 PASSER, X3 PASSER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

Commit message: updated schematics
Parts:
- IC2: value 24LC-I/OT -> 24LC32A
Changed lines of the file:
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@@
 <attribute name="NAME" x="31.4" y="31" size="0.8128" layer="21" font="vector" ratio="10" rot="R90" align="center"/>
 </element>
-<element name="IC2" library="we-chip" package="SOT23-5" value="24LC-I/OT" x="24.13" y="10.95375" smashed="yes" rot="MR270">
+<element name="IC2" library="we-chip" package="SOT23-5" value="24LC32A" x="24.13" y="10.95375" smashed="yes" rot="MR270">
 <attribute name="NAME" x="24.13" y="13.49375" size="0.8128" layer="26" font="vector" ratio="10" rot="MR180" align="center"/>
 <attribute name="VALUE" x="24.13" y="10.95375" size="0.8128" layer="28" font="vector" ratio="10" rot="MR180" align="center"/>
