File: pcb/RPi-Display_v10.sch (EAGLE design)
At the start: 42 parts, among them IC1 ADS7846, Q1 N-CHN, SW1 SW4S, U1 TS5204-3V3, X1 PASSER, X2 PASSER, X3 PASSER, X4 PASSER

Commit message: cleaned up schematics and layout
Changed lines of the file:
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@@
 <setting verticaltext="up"/>
 </settings>
-<grid distance="0.1" unitdist="inch" unit="inch" style="lines" multiple="1" display="no" altdistance="0.01" altunitdist="inch" altunit="inch"/>
+<grid distance="0.05" unitdist="inch" unit="inch" style="lines" multiple="1" display="yes" altdistance="0.025" altunitdist="inch" altunit="inch"/>
 <layers>
 <layer number="1" name="Top" color="4" fill="1" visible="no" active="no"/>
@@
 <part name="U$1" library="welectronic" deviceset="WE-LOGO" device="PLACE" value="WE-LOGO"/>
 <part name="LOGO1" library="OSHW" deviceset="OSHW_LOGO_6MIL" device="X0150-NT"/>
-<part name="FRAME1" library="frames" deviceset="A4L-LOC" device=""/>
 <part name="LCD1" library="Display" deviceset="MI0283QT9" device=""/>
 <part name="R1" library="rcl" deviceset="R-EU_" device="R0603" value="47"/>
@@
 <part name="+3V7" library="supply1" deviceset="+3V3" device=""/>
 <part name="P+5" library="supply1" deviceset="+5V" device=""/>
+<part name="FRAME1" library="we-symbol" deviceset="FRAME-A4L" device=""/>
 </parts>
 <sheets>
@@
 <text x="36.83" y="162.56" size="3.81" layer="250">2.8" Display with Touchpanel</text>
 <text x="180.34" y="162.56" size="3.81" layer="250">Raspberry Pi</text>
-<text x="161.29" y="31.75" size="1.27" layer="95">Released under the Creative Commons Attribution Share-Alike License</text>
-<text x="161.29" y="29.21" size="1.27" layer="95">http://creativecommons.org/licenses/by-sa/4.0/</text>
-<text x="161.29" y="25.4" size="1.27" layer="95">Designed by Andreas Watterott (Watterott electronic)</text>
+<text x="162.56" y="21.59" size="1.27" layer="95">Released under the Creative Commons Attribution Share-Alike License</text>
+<text x="162.56" y="19.05" size="1.27" layer="95">http://creativecommons.org/licenses/by-sa/4.0/</text>
+<text x="162.56" y="15.24" size="1.27" layer="95">Designed by Andreas Watterott (Watterott electronic)</text>
 <text x="128.27" y="100.33" size="3.81" layer="250">Touch Controller</text>
 <text x="139.7" y="59.69" size="1.778" layer="95">or TSC2046</text>
@@
 <attribute name="VALUE" x="107.315" y="7.493" size="1.778" layer="96"/>
 </instance>
-<instance part="X1" gate="G$1" x="167.64" y="17.78"/>
-<instance part="X2" gate="G$1" x="175.26" y="17.78"/>
-<instance part="X3" gate="G$1" x="182.88" y="17.78"/>
-<instance part="X4" gate="G$1" x="190.5" y="17.78"/>
-<instance part="U$1" gate="G$1" x="203.2" y="17.78"/>
-<instance part="LOGO1" gate="G$1" x="203.2" y="10.16"/>
-<instance part="FRAME1" gate="G$1" x="0" y="0" smashed="yes">
-<attribute name="DRAWING_NAME" x="217.17" y="15.24" size="2.54" layer="94" font="vector"/>
-<attribute name="LAST_DATE_TIME" x="217.17" y="10.16" size="2.286" layer="94" font="vector"/>
-<attribute name="SHEET" x="230.505" y="5.08" size="2.54" layer="94" font="vector"/>
-</instance>
+<instance part="X1" gate="G$1" x="165.1" y="7.62" smashed="yes"/>
+<instance part="X2" gate="G$1" x="170.18" y="7.62" smashed="yes"/>
+<instance part="X3" gate="G$1" x="175.26" y="7.62" smashed="yes"/>
+<instance part="X4" gate="G$1" x="180.34" y="7.62" smashed="yes"/>
+<instance part="U$1" gate="G$1" x="208.28" y="7.62"/>
+<instance part="LOGO1" gate="G$1" x="198.12" y="7.62"/>
 <instance part="LCD1" gate="G$1" x="71.12" y="100.33"/>
 <instance part="R1" gate="G$1" x="100.33" y="110.49" smashed="yes">
@@
 <attribute name="VALUE" x="203.835" y="101.6" size="1.778" layer="96" rot="R180"/>
 </instance>
+<instance part="FRAME1" gate="G$1" x="0" y="0"/>
 </instances>
 <busses>
