File: pcb/GPIO-Adapter_v10.sch (EAGLE design)
At the start: 8 parts, among them J1 FPC40_PIN, X1 PASSER, X2 PASSER, X3 PASSER, X4 PASSER

Commit message: cleaned up schematics and layout
Changed lines of the file:
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@@
 <setting verticaltext="up"/>
 </settings>
-<grid distance="0.1" unitdist="inch" unit="inch" style="lines" multiple="1" display="no" altdistance="0.01" altunitdist="inch" altunit="inch"/>
+<grid distance="0.05" unitdist="inch" unit="inch" style="lines" multiple="1" display="yes" altdistance="0.025" altunitdist="inch" altunit="inch"/>
 <layers>
 <layer number="1" name="Top" color="4" fill="1" visible="no" active="no"/>
@@
 <part name="X4" library="SMD" deviceset="PASSER" device=""/>
 <part name="LOGO1" library="OSHW" deviceset="OSHW_LOGO_6MIL" device="X0150-NT"/>
-<part name="FRAME1" library="frames" deviceset="A4L-LOC" device=""/>
 <part name="RPI" library="we-board" deviceset="RPI_B+" device="-CON" value="RPI"/>
 <part name="J1" library="we-con" deviceset="FPC40_PIN" device=""/>
 <part name="LOGO2" library="we-symbol" deviceset="LOGO" device="-S_PLACE_M" value="LOGO-S_PLACE_M"/>
+<part name="FRAME1" library="we-symbol" deviceset="FRAME-A4L" device=""/>
 </parts>
 <sheets>
 <sheet>
 <plain>
-<text x="161.29" y="31.75" size="1.27" layer="95">Released under the Creative Commons Attribution Share-Alike License</text>
-<text x="161.29" y="29.21" size="1.27" layer="95">http://creativecommons.org/licenses/by-sa/4.0/</text>
-<text x="161.29" y="25.4" size="1.27" layer="95">Designed by Andreas Watterott (Watterott electronic)</text>
+<text x="162.56" y="21.59" size="1.27" layer="95">Released under the Creative Commons Attribution Share-Alike License</text>
+<text x="162.56" y="19.05" size="1.27" layer="95">http://creativecommons.org/licenses/by-sa/4.0/</text>
+<text x="162.56" y="15.24" size="1.27" layer="95">Designed by Andreas Watterott (Watterott electronic)</text>
 </plain>
 <instances>
-<instance part="X1" gate="G$1" x="167.64" y="19.05"/>
-<instance part="X2" gate="G$1" x="175.26" y="19.05"/>
-<instance part="X3" gate="G$1" x="182.88" y="19.05"/>
-<instance part="X4" gate="G$1" x="190.5" y="19.05"/>
-<instance part="LOGO1" gate="G$1" x="207.01" y="11.43"/>
-<instance part="FRAME1" gate="G$1" x="0" y="0" smashed="yes">
-<attribute name="DRAWING_NAME" x="217.17" y="15.24" size="2.54" layer="94" font="vector"/>
-<attribute name="LAST_DATE_TIME" x="217.17" y="10.16" size="2.286" layer="94" font="vector"/>
-<attribute name="SHEET" x="230.505" y="5.08" size="2.54" layer="94" font="vector"/>
-</instance>
+<instance part="X1" gate="G$1" x="165.1" y="7.62"/>
+<instance part="X2" gate="G$1" x="170.18" y="7.62"/>
+<instance part="X3" gate="G$1" x="175.26" y="7.62"/>
+<instance part="X4" gate="G$1" x="180.34" y="7.62"/>
+<instance part="LOGO1" gate="G$1" x="198.12" y="7.62"/>
 <instance part="RPI" gate="RPI" x="128.27" y="99.06"/>
-<instance part="LOGO2" gate="G$1" x="207.01" y="19.05"/>
+<instance part="LOGO2" gate="G$1" x="208.28" y="7.62"/>
 <instance part="J1" gate="P40" x="148.59" y="73.66"/>
 <instance part="J1" gate="P1" x="107.95" y="121.92" rot="R180"/>
@@
 <instance part="J1" gate="P38" x="148.59" y="76.2"/>
 <instance part="J1" gate="P39" x="107.95" y="73.66" rot="R180"/>
+<instance part="FRAME1" gate="G$1" x="0" y="0"/>
 </instances>
 <busses>
