File: pcb/RPi-Display_Bplus_v11.brd (EAGLE design)
At the start: 69.5 x 56 mm, 59 parts, among them IC1 ADS7846, IC2 24LC32A, IC3 LDO-TS9011-3V3, Q1 N-CHN, SW1 SWITCH-PTS840P, SW2 SWITCH-PTS840P, SW3 SWITCH-PTS840P, X1 PASSER, X2 PASSER, X3 PASSER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

Commit message: updated layout and schematics
Parts:
- 3V3-VREF, IO24-RS, MISO, MOSI, SCK, WP: value JUMPER2-NOCREAM -> JUMPER2-0603-NC; device we-rcl:JUMPER2_NC -> we-rcl:JUMPER2-0603_NC
- 5V-3V3, BL, IM0, IM1: value JUMPER3-NOCREAM -> JUMPER3-0603-NC; device we-rcl:JUMPER3_NC -> we-rcl:JUMPER3-0603_NC
- IC2: value 24LC32A -> 24LC-I/OT
- LOGO2: value WEEE_LOGO -> WEEE_LOGO-M; device we-symbol:WEEE -> we-symbol:WEEE_TPLAC_M
- RPI: device we-board:RPI_B+ -> we-board:RPI-B+_CON
- SW1, SW2, SW3: value SWITCH-PTS840P -> SW-TACTILE-PTS840P
Connections:
- net GND: now also SW1.3, SW1.4, SW2.3, SW2.4, SW3.3, SW3.4; no longer SW1.1, SW1.2, SW2.1, SW2.2, SW3.1, SW3.2
- net IO17: now also SW1.1, SW1.2; no longer SW1.3, SW1.4
- net IO22: now also SW3.1, SW3.2; no longer SW3.3, SW3.4
- net IO27: now also SW2.1, SW2.2; no longer SW2.3, SW2.4
Routing:
- net GND: track 44.2 -> 64.0 mm
- net IO22: track 98.3 -> 96.8 mm
- net IO17: track 70.4 -> 68.9 mm
- net IO27: track 83.8 -> 82.4 mm
