File: hardware/RPi-Display_Bplus_v11.brd (EAGLE design)
At the start: 69.5 x 56 mm, 59 parts, among them IC1 ADS7846, IC2 24LC-I/OT, IC3 LDO-TS9011-3V3, Q1 N-CHN, SW1 SW-TACTILE-PTS840P, SW2 SW-TACTILE-PTS840P, SW3 SW-TACTILE-PTS840P, X1 PASSER, X2 PASSER, X3 PASSER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

Commit message: updated docu and schematics
Other:
- board text added: "Top Contacts"
Changed lines of the file:
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@@
 <?xml version="1.0" encoding="utf-8"?>
 <!DOCTYPE eagle SYSTEM "eagle.dtd">
-<eagle version="7.3.0">
+<eagle version="7.5.0">
 <drawing>
 <settings>
@@
 <text x="14.76375" y="46.0375" size="0.889" layer="26" font="vector" ratio="10" rot="MR0">18</text>
 <text x="11.90625" y="46.0375" size="0.889" layer="26" font="vector" ratio="10" rot="MR0">12</text>
+<text x="17.78" y="39.37" size="0.8128" layer="21" font="vector" ratio="14" align="center">Top Contacts</text>
 </plain>
 <attributes>
