File: hardware/RPi-Display_v10.brd (EAGLE design)
At the start: 85 x 56 mm, 42 parts, among them IC1 ADS7846, Q1 N-CHN, SW1 SW4S, U1 TS5204-3V3, X1 PASSER, X2 PASSER, X3 PASSER, X4 PASSER

Commit message: updated schematics
Parts:
- C1, C4: value 1uF -> 2uF
Changed lines of the file:
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@@
 <layer number="51" name="tDocu" color="7" fill="1" visible="yes" active="yes"/>
 <layer number="52" name="bDocu" color="7" fill="1" visible="yes" active="yes"/>
-<layer number="53" name="tCopper" color="7" fill="11" visible="no" active="no"/>
-<layer number="54" name="bCopper" color="7" fill="1" visible="no" active="no"/>
-<layer number="56" name="wert" color="7" fill="1" visible="no" active="no"/>
 <layer number="91" name="Nets" color="2" fill="1" visible="no" active="no"/>
 <layer number="92" name="Busses" color="1" fill="1" visible="no" active="no"/>
@@
 <layer number="97" name="Info" color="7" fill="1" visible="no" active="no"/>
 <layer number="98" name="Guide" color="6" fill="1" visible="no" active="no"/>
-<layer number="100" name="Muster" color="7" fill="1" visible="no" active="no"/>
-<layer number="217" name="217bmp" color="18" fill="1" visible="no" active="no"/>
-<layer number="218" name="218bmp" color="19" fill="1" visible="no" active="no"/>
-<layer number="219" name="219bmp" color="20" fill="1" visible="no" active="no"/>
-<layer number="220" name="220bmp" color="21" fill="1" visible="no" active="no"/>
-<layer number="221" name="221bmp" color="22" fill="1" visible="no" active="no"/>
-<layer number="222" name="222bmp" color="23" fill="1" visible="no" active="no"/>
-<layer number="223" name="223bmp" color="24" fill="1" visible="no" active="no"/>
-<layer number="224" name="224bmp" color="25" fill="1" visible="no" active="no"/>
-<layer number="251" name="SMDround" color="12" fill="11" visible="no" active="no"/>
 </layers>
 <board>
@@
 <attribute name="VALUE" x="57.4675" y="15.39875" size="0.8128" layer="28" font="vector" rot="MR90"/>
 </element>
-<element name="C1" library="rcl" package="C0603" value="1uF" x="62.3888" y="13.335" smashed="yes" rot="MR270">
+<element name="C1" library="rcl" package="C0603" value="2uF" x="62.3888" y="13.335" smashed="yes" rot="MR270">
 <attribute name="NAME" x="61.75375" y="11.58875" size="0.8128" layer="26" font="vector" ratio="10" rot="MR180"/>
 <attribute name="VALUE" x="62.07125" y="15.08125" size="0.8128" layer="28" font="vector" rot="MR90"/>
@@
 <attribute name="VALUE" x="50.8" y="15.08125" size="0.8128" layer="28" font="vector" rot="MR90"/>
 </element>
-<element name="C4" library="rcl" package="C0603" value="1uF" x="53.1811" y="13.335" smashed="yes" rot="MR270">
+<element name="C4" library="rcl" package="C0603" value="2uF" x="53.1811" y="13.335" smashed="yes" rot="MR270">
 <attribute name="NAME" x="52.3875" y="11.58875" size="0.8128" layer="26" font="vector" rot="MR180"/>
 <attribute name="VALUE" x="52.86375" y="15.08125" size="0.8128" layer="28" font="vector" rot="MR90"/>
